File: Homework 2/PIC32/PIC32.brd (EAGLE design)
At the start: 100 x 100 mm, 23 parts

Commit message: Design change
Parts:
- moved LED1 94.6 mm to (7.87, 32.9), turned to 90 degrees
- moved J1 87.0 mm to (5.08, 5.08), turned to 270 degrees
- moved R1 86.1 mm to (11.4, 33.0)
- moved C3 83.6 mm to (20.3, 10.2), turned to 180 degrees
- moved C4 81.6 mm to (20.3, 3.81), turned to 180 degrees
- moved C5 73.6 mm to (12.7, 19.1), turned to 180 degrees
- moved U$3 71.9 mm to (5.08, 25.4), turned to 0 degrees
- moved U$2 68.6 mm to (3.81, 15.2)
- moved U$4 59.7 mm to (94.0, 7.62), turned to 270 degrees
- moved U$5 54.6 mm to (94.0, 38.1), turned to 270 degrees
- moved U$9 53.0 mm to (97.8, 20.3), turned to 90 degrees
- moved R2 51.1 mm to (91.4, 44.5)
- moved R3 43.3 mm to (88.9, 10.2), turned to 90 degrees
- moved LED2 39.8 mm to (86.4, 38.1)
- moved R4 29.2 mm to (91.4, 50.8)
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Routing:
- net +3V3: track 0.00 -> 208.2 mm, vias 0 -> 3
- net +5V: track 0.00 -> 107.1 mm, vias 0 -> 1
- net USBID: track 0.00 -> 100.4 mm, vias 0 -> 2
- net MCLR: track 0.00 -> 84.4 mm
- net D-: track 0.00 -> 62.8 mm, vias 0 -> 2
- net D+: track 0.00 -> 62.3 mm, vias 0 -> 2
- net PGD: track 0.00 -> 56.0 mm, vias 0 -> 2
- net B4: track 0.00 -> 53.9 mm
- net PGC: track 0.00 -> 53.4 mm, vias 0 -> 2
- net A4: track 0.00 -> 48.2 mm, vias 0 -> 1
- net GND: track 0.00 -> 42.1 mm, vias 0 -> 1
- net A0: track 0.00 -> 34.7 mm
- net A1: track 0.00 -> 34.3 mm
- net B15: track 0.00 -> 33.9 mm
- net B14: track 0.00 -> 33.0 mm
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- added copper zone on layer 16, net GND
Other:
- board text added: "+"
- board text added: "3.3V"
- board text added: "4/10/2019"
- board text added: "5V"
- board text added: "A0"
- board text added: "A1"
- board text added: "A4"
- board text added: "B13"
- board text added: "B14"
- board text added: "B15"
- board text added: "B2"
- board text added: "B3"
- board text added: "B4"
- board text added: "B7"
- board text added: "B8"
- board text added: "B9"
- board text added: "GND"
- board text added: "JOSHUA CHO"
- board text added: "ME433 SPRING 2019"
